File: HE75/HE75.kicad_pcb (KiCad board)
At the start: 2 copper layers, 284.7 x 94.2 mm, 351 parts, among them J1 TYPE-C-31-M-12, J2 JST_SH, SW1 TS-1187A-B-A-B, SW2 TS-1187A-B-A-B, U1 USBLC6-2SC6, U2 TLV75733PDBV, U3 XC6206P332MR-G, U4 AT32F405RCT7, Y1 X322512MSB4SI

Commit message: First working revision
Connected all traces
Parts:
- removed the C173 at (199.0, 71.3)
- C161, C162, C163: moved to B.Cu
- moved C162 262.2 mm to (252.6, 78.9), turned to -90 degrees
- moved C163 192.6 mm to (183.1, 84.4), turned to 90 degrees
- moved C161 187.4 mm to (177.8, 84.4), turned to -90 degrees
- moved AM10 67.7 mm to (256.2, 75.7)
- moved AM9 23.7 mm to (189.8, 75.5)
- moved C147 23.5 mm to (186.0, 78.7)
- moved C164 19.1 mm to (196.9, 84.4)
- moved C168 19.1 mm to (235.0, 84.4)
- moved C170 19.1 mm to (254.1, 84.4)
- moved C172 19.1 mm to (273.1, 84.4)
- moved C166 19.0 mm to (215.9, 84.4)
- moved C169 19.0 mm to (240.2, 84.4)
- moved C154 17.9 mm to (12.0, 29.1), turned to -135 degrees
- moved C167 17.9 mm to (219.8, 82.4), turned to 0 degrees
- moved C171 17.8 mm to (257.9, 82.4), turned to 0 degrees
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Connections:
- AM1 pad 12: HE1 -> HE4
- AM1 pad 13: HE4 -> HE3
- AM1 pad 14: HE3 -> HE2
- AM1 pad 15: HE2 -> HE1
- AM10 pad 1: unconnected-(AM10-X4-Pad1) -> HE58
- AM10 pad 12: unconnected-(AM10-X3-Pad12) -> GND
- AM10 pad 13: unconnected-(AM10-X0-Pad13) -> HE75
- AM10 pad 14: unconnected-(AM10-X1-Pad14) -> HE74
- AM10 pad 15: unconnected-(AM10-X2-Pad15) -> HE73
- AM10 pad 2: unconnected-(AM10-X6-Pad2) -> HE59
- AM10 pad 4: unconnected-(AM10-X7-Pad4) -> HE60
- AM10 pad 5: unconnected-(AM10-X5-Pad5) -> GND
- AM3 pad 12: HE16 -> HE19
- AM3 pad 13: HE19 -> HE18
- AM3 pad 14: HE18 -> HE17
- AM3 pad 15: HE17 -> HE16
- AM6 pad 12: HE55 -> GND
- AM6 pad 13: HE56 -> HE45
- AM6 pad 14: HE57 -> HE44
- AM7 pad 1: unconnected-(AM7-X4-Pad1) -> HE46
- AM7 pad 12: HE61 -> HE64
- AM7 pad 13: HE60 -> HE63
- AM7 pad 14: HE59 -> HE62
- AM7 pad 15: HE58 -> HE61
- AM7 pad 2: HE44 -> HE47
- AM7 pad 4: HE45 -> HE48
- AM7 pad 5: HE46 -> HE49
- AM8 pad 1: HE47 -> HE50
- AM8 pad 12: HE62 -> HE68
- AM8 pad 13: HE63 -> HE67
- AM8 pad 14: HE64 -> HE66
- AM8 pad 2: HE48 -> HE51
- AM8 pad 4: HE49 -> HE52
- AM8 pad 5: HE50 -> HE53
- AM9 pad 1: HE51 -> HE54
- AM9 pad 12: HE66 -> HE72
- AM9 pad 13: HE67 -> HE71
- AM9 pad 14: HE68 -> HE70
- AM9 pad 2: HE52 -> HE55
- AM9 pad 4: HE53 -> HE56
- AM9 pad 5: HE54 -> HE57
Routing:
- net +3.3VA: track 1.47 -> 2061.9 mm, vias 0 -> 12
- net MUX_SELECT_2: track 0.00 -> 494.5 mm, vias 0 -> 9
- net MUX_SELECT_1: track 0.00 -> 488.8 mm, vias 0 -> 9
- net MUX_SELECT_0: track 0.00 -> 486.7 mm, vias 0 -> 9
- net MUX_OUT_10: track 0.00 -> 266.2 mm, vias 0 -> 2
- net MUX_OUT_9: track 0.00 -> 189.3 mm, vias 0 -> 2
- net MUX_OUT_6: track 0.00 -> 160.6 mm, vias 0 -> 2
- net MUX_OUT_4: track 0.00 -> 154.1 mm, vias 0 -> 2
- net MUX_OUT_2: track 0.00 -> 152.0 mm, vias 0 -> 2
- net GND: track 0.00 -> 129.1 mm, vias 0 -> 264
- net HE45: track 0.00 -> 116.8 mm
- net MUX_OUT_8: track 0.00 -> 112.9 mm, vias 0 -> 2
- net MUX_OUT_1: track 0.00 -> 105.1 mm, vias 0 -> 2
- net +3.3V: track 0.00 -> 101.5 mm, vias 0 -> 3
- net HE44: track 0.00 -> 98.6 mm
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