File: HE75/HE75.kicad_sch (KiCad schematic)
At the start: 331 parts, among them J1 TYPE-C-31-M-12, J2 JST_SH, SW1 TS-1187A-B-A-B, SW2 TS-1187A-B-A-B, U1 USBLC6-2SC6, U2 TLV75733PDBV, U3 XC6206P332MR-G, U4 AT32F405RCT7, Y1 X322512MSB4SI

Commit message: Modified PCB
Changed switch locations, added components to support higher switch count, removed conflicting mounting holes
Parts:
- removed MX76: 1.25U, HE60:MX-1.25U, symbol Mechanical:MountingHole
- added AM10: SN74LV4051A, Package_SO:TSSOP-16_4.4x5mm_P0.65mm, symbol 4xxx:4051
- added C161, C162, C164, C166, C168, C170, C172: 100n, Capacitor_SMD:C_0402_1005Metric, symbol Device:C
- added C163, C165, C167, C169, C171, C173: 4.7n, Capacitor_SMD:C_0402_1005Metric, symbol Device:C
- added HE70, HE71, HE72, HE73, HE74, HE75: MT9102ET, Package_TO_SOT_SMD:SOT-23-3, symbol HE60:MT9102ET
- MX15: value 2U -> 1U; footprint HE60:MX-2U -> HE60:MX-1U
- MX17, MX30, MX59, MX63, MX71, MX75: value 1.5U -> 1U; footprint HE60:MX-1.5U -> HE60:MX-1U
- MX31, MX55: value 1.75U -> 1U; footprint HE60:MX-1.75U -> HE60:MX-1U
- MX43, MX44: value 2.25U -> 1U; footprint HE60:MX-2.25U -> HE60:MX-1U
- MX56: value 2.75U -> 1U; footprint HE60:MX-2.75U -> HE60:MX-1U
- MX58, MX60, MX62, MX70, MX72, MX74: value 1.25U -> 1U; footprint HE60:MX-1.25U -> HE60:MX-1U
- MX65: value 2.25U -> 1U; footprint HE60:MX-2.25U-ReversedStabilizers -> HE60:MX-1U
- MX66: value 6.25U -> 1U; footprint HE60:MX-6.25U-ReversedStabilizers -> HE60:MX-1U
- MX67: value 7U -> 1U; footprint HE60:MX-7U-ReversedStabilizers -> HE60:MX-1U
- MX68: value 2.75U -> 1U; footprint HE60:MX-2.75U-ReversedStabilizers -> HE60:MX-1U
Connections:
- net +3.3VA: now also AM10.16 (VDD), C161.1, C162.1, C164.1, C166.1, C168.1, C170.1, C172.1, HE70.1 (VCC), HE71.1 (VCC), HE72.1 (VCC), HE73.1 (VCC), HE74.1 (VCC), HE75.1 (VCC)
- net GND: now also AM2.12 (X3), AM10.6 (Inh), AM10.7 (VEE), AM10.8 (VSS), C161.2, C162.2, C163.2, C164.2, C165.2, C166.2, C167.2, C168.2, C169.2, C170.2, C171.2, C172.2, C173.2, HE70.3 (GND), HE71.3 (GND), HE72.3 (GND), HE73.3 (GND), HE74.3 (GND), HE75.3 (GND); no longer AM1.12 (X3), AM5.15 (X2)
- net HE1: now also AM1.12 (X3); no longer AM3.15 (X2)
- net HE16: now also AM3.12 (X3); no longer AM2.12 (X3)
- net HE17: now also AM3.15 (X2); no longer AM3.14 (X1)
- net HE18: now also AM3.14 (X1); no longer AM3.13 (X0)
- net HE19: now also AM3.13 (X0); no longer AM3.12 (X3)
- net HE31: now also AM5.15 (X2); no longer AM7.1 (X4)
- net MUX_SELECT_0: now also AM10.11 (A)
- net MUX_SELECT_1: now also AM10.10 (B)
- net MUX_SELECT_2: now also AM10.9 (C)
- net MUX_OUT_10: now reaches U4.16 (PA2)
- net MUX_OUT_10: now also AM10.3 (X)
- new net HE70: C163.1, HE70.2 (OUT)
- new net HE71: C165.1, HE71.2 (OUT)
- new net HE72: C167.1, HE72.2 (OUT)
- new net HE73: C169.1, HE73.2 (OUT)
- new net HE74: C171.1, HE74.2 (OUT)
- new net HE75: C173.1, HE75.2 (OUT)
- no-connect marks 41 -> 40
Other:
- moved on the sheet: C31, C32, HE16

Commit message: First working revision
Connected all traces
Connections:
- net GND: now also AM10.12 (X3), AM10.5 (X5), AM6.12 (X3)
- net HE1: now also AM1.15 (X2); no longer AM1.12 (X3)
- net HE16: now also AM3.15 (X2); no longer AM3.12 (X3)
- net HE17: now also AM3.14 (X1); no longer AM3.15 (X2)
- net HE18: now also AM3.13 (X0); no longer AM3.14 (X1)
- net HE19: now also AM3.12 (X3); no longer AM3.13 (X0)
- net HE2: now also AM1.14 (X1); no longer AM1.15 (X2)
- net HE3: now also AM1.13 (X0); no longer AM1.14 (X1)
- net HE4: now also AM1.12 (X3); no longer AM1.13 (X0)
- net HE44: now also AM6.14 (X1); no longer AM7.2 (X6)
- net HE45: now also AM6.13 (X0); no longer AM7.4 (X7)
- net HE46: now also AM7.1 (X4); no longer AM7.5 (X5)
- net HE47: now also AM7.2 (X6); no longer AM8.1 (X4)
- net HE48: now also AM7.4 (X7); no longer AM8.2 (X6)
- net HE49: now also AM7.5 (X5); no longer AM8.4 (X7)
- net HE50: now also AM8.1 (X4); no longer AM8.5 (X5)
- net HE51: now also AM8.2 (X6); no longer AM9.1 (X4)
- net HE52: now also AM8.4 (X7); no longer AM9.2 (X6)
- net HE53: now also AM8.5 (X5); no longer AM9.4 (X7)
- net HE54: now also AM9.1 (X4); no longer AM9.5 (X5)
- net HE55: now also AM9.2 (X6); no longer AM6.12 (X3)
- net HE56: now also AM9.4 (X7); no longer AM6.13 (X0)
- net HE57: now also AM9.5 (X5); no longer AM6.14 (X1)
- net HE58: now also AM10.1 (X4); no longer AM7.15 (X2)
- net HE59: now also AM10.2 (X6); no longer AM7.14 (X1)
- net HE60: now also AM10.4 (X7); no longer AM7.13 (X0)
- net HE61: now also AM7.15 (X2); no longer AM7.12 (X3)
- net HE62: now also AM7.14 (X1); no longer AM8.12 (X3)
- net HE63: now also AM7.13 (X0); no longer AM8.13 (X0)
- net HE64: now also AM7.12 (X3); no longer AM8.14 (X1)
- net HE66: now also AM8.14 (X1); no longer AM9.12 (X3)
- net HE67: now also AM8.13 (X0); no longer AM9.13 (X0)
- net HE68: now also AM8.12 (X3); no longer AM9.14 (X1)
- net HE70: now also AM9.14 (X1)
- net HE71: now also AM9.13 (X0)
- net HE72: now also AM9.12 (X3)
- net HE73: now also AM10.15 (X2)
- net HE74: now also AM10.14 (X1)
- net HE75: now also AM10.13 (X0)
